Commit message: added camera, lidar, base gazebo farming world

File: urdf/robot.urdf.xacro (robot description, xacro)
@@ -7,3 +7,4 @@
     <xacro:include filename="$(find agri_bot)/urdf/gazebo_control.xacro" />
     <xacro:include filename="$(find agri_bot)/urdf/s_camera.xacro" />
+    <xacro:include filename="$(find agri_bot)/urdf/s_lidar.xacro" />
 </robot>

File: urdf/robot_core.urdf.xacro (robot description, xacro)
@@ -49,5 +49,5 @@
 </link>
 <gazebo reference="front_right_wheel">
-    <material>Gazebo/Blue</material>
+    <material>Gazebo/Black</material>
 </gazebo>
 <link name="front_left_wheel">
@@ -69,5 +69,5 @@
 </link>
 <gazebo reference="front_left_wheel">
-    <material>Gazebo/Blue</material>
+    <material>Gazebo/Black</material>
 </gazebo>
 <link name="rear_right_wheel">
@@ -89,5 +89,5 @@
 </link>
 <gazebo reference="rear_right_wheel">
-    <material>Gazebo/Blue</material>
+    <material>Gazebo/Black</material>
 </gazebo>
 <link name="rear_left_wheel">
@@ -109,5 +109,5 @@
 </link>
 <gazebo reference="rear_left_wheel">
-    <material>Gazebo/Blue</material>
+    <material>Gazebo/Black</material>
 </gazebo>
 <joint name="base_to_chassis" type="fixed">

File: urdf/s_camera.xacro (robot description, xacro)
@@ -1,52 +1,13 @@
 <?xml version="1.0"?>
 <robot xmlns:xacro="http://www.ros.org/wiki/xacro" >
-    <joint name="camera_joint" type="fixed">
-        <parent link="chassis_link"/>
-        <child link="camera_link"/>
-        <origin xyz="0.06 0 0.14" rpy="0 0 0"/>
-    </joint>
-    <link name="camera_link">
-        <visual>
-            <geometry>
-                <box size="0.010 0.03 0.03"/>
-            </geometry>
-            <material name="black"/>
-        </visual>
-        <visual>
-            <origin xyz="0 0 -0.05"/>
-            <geometry>
-                <cylinder radius="0.002" length="0.1"/>
-            </geometry>
-            <material name="black"/>
-        </visual>
-    </link>
-    <joint name="camera_optical_joint" type="fixed">
-        <parent link="camera_link"/>
-        <child link="camera_link_optical"/>
-        <origin xyz="0 0 0" rpy="${-pi/2} 0 ${-pi/2}"/>
-    </joint>
-    <link name="camera_link_optical"></link>
-    <gazebo reference="camera_link">
-        <material>Gazebo/Black</material>
-        <sensor name="camera" type="camera">
-            <pose> 0 0 0 0 0 0 </pose>
-            <visualize>true</visualize>
-            <update_rate>10</update_rate>
-            <camera>
-                <horizontal_fov>1.089</horizontal_fov>
-                <image>
-                    <format>R8G8B8</format>
-                    <width>640</width>
-                    <height>480</height>
-                </image>
-                <clip>
-                    <near>0.05</near>
-                    <far>8.0</far>
-                </clip>
-            </camera>
-            <plugin name="camera_controller" filename="libgazebo_ros_camera.so">
-                <frame_name>camera_link_optical</frame_name>
-            </plugin>
-        </sensor>
-    </gazebo>
+<xacro:include filename="$(find agri_bot)/urdf/camera_macro.xacro"/>
+<xacro:property name="camera_x" value="0.00"/>
+<xacro:property name="camera_y" value="0.14"/>
+<xacro:property name="camera_z" value="0.07"/>
+<xacro:camera_create name = "left">
+    <origin xyz="${camera_x} ${-camera_y} ${camera_z}" rpy="0 0 ${-pi/2}"/>
+</xacro:camera_create>
+<xacro:camera_create name = "right">
+    <origin xyz="${camera_x} ${camera_y} ${camera_z}" rpy="0 0 ${pi/2}"/>
+</xacro:camera_create>
 </robot>
