Commit message: fixed gazebo plugins, frames need to be rearranged

File: urdf/gazebo_control.xacro (robot description, xacro)
@@ -1,22 +1,23 @@
 <?xml version="1.0"?>
 <robot xmlns:xacro="http://www.ros.org/wiki/xacro">
-    <gazebo>
-        <plugin name="diff_drive" filename="libgazebo_ros_diff_drive.so">
-            <left_joint>left_wheel_joint</left_joint>
-            <right_joint>right_wheel_joint</right_joint>
-            <wheel_separation>0.32</wheel_separation>
-            <wheel_diameter>0.07</wheel_diameter>
-            <left_joint>left_wheel_joint</left_joint>
-            <right_joint>right_wheel_joint</right_joint>
-            <wheel_separation>0.32</wheel_separation>
-            <wheel_diameter>0.07</wheel_diameter>
-            <max_wheel_torque>200</max_wheel_torque>
-            <max_wheel_acceleration>10.0</max_wheel_acceleration>
-            <odometry_frame>odom</odometry_frame>
-            <robot_base_frame>base_link</robot_base_frame>
-            <publish_odom>true</publish_odom>
-            <publish_odom_tf>true</publish_odom_tf>
-            <publish_wheel_tf>true</publish_wheel_tf>
-        </plugin>
-    </gazebo>
+<gazebo>
+    <plugin name="skid_steer_controller" filename="libgazebo_ros_diff_drive.so">
+        <num_wheel_pairs>2</num_wheel_pairs>
+        <left_joint>fl_to_chassis</left_joint>
+        <right_joint>fr_to_chassis</right_joint>
+        <left_joint>rl_to_chassis</left_joint>
+        <right_joint>rr_to_chassis</right_joint>
+        <wheel_separation>0.375</wheel_separation>
+        <wheel_separation>0.375</wheel_separation>
+        <wheel_diameter>0.2</wheel_diameter>
+        <wheel_diameter>0.2</wheel_diameter>
+        <max_wheel_torque>200</max_wheel_torque>
+        <max_wheel_acceleration>10.0</max_wheel_acceleration>
+        <odometry_frame>odom</odometry_frame>
+        <robot_base_frame>base_link</robot_base_frame>
+        <publish_odom>true</publish_odom>
+        <publish_odom_tf>true</publish_odom_tf>
+        <publish_wheel_tf>true</publish_wheel_tf>
+    </plugin>
+</gazebo>
 </robot>

File: urdf/robot.urdf.xacro (robot description, xacro)
@@ -1,4 +1,4 @@
 <?xml version="1.0" ?>
-<robot name="agro_bot" xmlns:xacro="http://www.ros.org/wiki/xacro" >
+<robot name="agri_bot" xmlns:xacro="http://www.ros.org/wiki/xacro" >
     <xacro:arg name="use_ros2_control" default="true"/>
     <xacro:arg name="sim_mode" default="false"/>

File: urdf/robot_core.urdf.xacro (robot description, xacro)
@@ -28,4 +28,7 @@
     </xacro:inertial_box>
 </link>
+<gazebo reference="chassis_link">
+    <material>Gazebo/Blue</material>
+</gazebo>
 <link name="front_right_wheel">
     <visual>
@@ -45,4 +48,7 @@
     </xacro:inertial_cylinder>
 </link>
+<gazebo reference="front_right_wheel">
+    <material>Gazebo/Blue</material>
+</gazebo>
 <link name="front_left_wheel">
     <visual>
@@ -62,4 +68,7 @@
     </xacro:inertial_cylinder>
 </link>
+<gazebo reference="front_left_wheel">
+    <material>Gazebo/Blue</material>
+</gazebo>
 <link name="rear_right_wheel">
     <visual>
@@ -79,4 +88,7 @@
     </xacro:inertial_cylinder>
 </link>
+<gazebo reference="rear_right_wheel">
+    <material>Gazebo/Blue</material>
+</gazebo>
 <link name="rear_left_wheel">
     <visual>
@@ -96,4 +108,7 @@
     </xacro:inertial_cylinder>
 </link>
+<gazebo reference="rear_left_wheel">
+    <material>Gazebo/Blue</material>
+</gazebo>
 <joint name="base_to_chassis" type="fixed">
     <parent link="base_link"/>
@@ -109,5 +124,5 @@
     <parent link="chassis_link"/>
     <child link="front_left_wheel"/>
-    <origin xyz = "${chassis_length/2 - chassis_length/8} -${chassis_width - 0.1} -${chassis_height/2}" rpy= "${pi/2} 0 0"/>
+    <origin xyz = "${chassis_length/2 - chassis_length/8} -${chassis_width - 0.1} -${chassis_height/2}" rpy= "-${pi/2} 0 0"/>
     <axis xyz="0 0 1"/>
 </joint>
@@ -121,5 +136,5 @@
     <parent link="chassis_link"/>
     <child link="rear_left_wheel"/>
-    <origin xyz = "-${chassis_length/2 - chassis_length/8} -${chassis_width - 0.1} -${chassis_height/2}" rpy= "${pi/2} 0 0"/>
+    <origin xyz = "-${chassis_length/2 - chassis_length/8} -${chassis_width - 0.1} -${chassis_height/2}" rpy= "-${pi/2} 0 0"/>
     <axis xyz="0 0 1"/>
 </joint>

Commit message: added nav and localization, added ekf files to be tested, in spot rotation has to be fixed

File: urdf/gazebo_control.xacro (robot description, xacro)
@@ -8,6 +8,6 @@
         <left_joint>rl_to_chassis</left_joint>
         <right_joint>rr_to_chassis</right_joint>
-        <wheel_separation>0.375</wheel_separation>
-        <wheel_separation>0.375</wheel_separation>
+        <wheel_separation>0.2</wheel_separation>
+        <wheel_separation>0.2</wheel_separation>
         <wheel_diameter>0.2</wheel_diameter>
         <wheel_diameter>0.2</wheel_diameter>

File: urdf/robot.urdf.xacro (robot description, xacro)
@@ -8,3 +8,5 @@
     <xacro:include filename="$(find agri_bot)/urdf/s_camera.xacro" />
     <xacro:include filename="$(find agri_bot)/urdf/s_lidar.xacro" />
+    <xacro:include filename="$(find agri_bot)/urdf/s_gps.xacro" />
+    <xacro:include filename="$(find agri_bot)/urdf/s_imu.xacro" />
 </robot>

File: urdf/robot_core.urdf.xacro (robot description, xacro)
@@ -10,5 +10,13 @@
 <xacro:property name="wheel_thickness" value = "0.1"/>
 <xacro:property name="wheel_mass"      value = "0.1"/>
+<xacro:property name="wheel_offset_y"  value = "0.2"/>
 <link name="base_link"/>
+<joint name="base_footprint_joint" type="fixed">
+    <parent link="base_link"/>
+    <child link="base_footprint"/>
+    <origin xyz="0 0 0" rpy="0 0 0"/>
+</joint>
+<link name="base_footprint">
+</link>
 <link name="chassis_link">
     <visual>
@@ -118,5 +126,5 @@
     <parent link="chassis_link"/>
     <child link="front_right_wheel"/>
-    <origin xyz = "${chassis_length/2 - chassis_length/8} ${chassis_width - 0.1} -${chassis_height/2}" rpy= "${pi/2} 0 0"/>
+    <origin xyz = "${chassis_length/2 - chassis_length/8} -${wheel_offset_y} -${chassis_height/2}" rpy= "${pi/2} 0 0"/>
     <axis xyz="0 0 1"/>
 </joint>
@@ -124,11 +132,11 @@
     <parent link="chassis_link"/>
     <child link="front_left_wheel"/>
-    <origin xyz = "${chassis_length/2 - chassis_length/8} -${chassis_width - 0.1} -${chassis_height/2}" rpy= "-${pi/2} 0 0"/>
-    <axis xyz="0 0 1"/>
+    <origin xyz = "${chassis_length/2 - chassis_length/8}  ${wheel_offset_y} -${chassis_height/2}" rpy= "-${pi/2} 0 0"/>
+    <axis xyz="0 0 -1"/>
 </joint>
 <joint name="rr_to_chassis" type="continuous">
     <parent link="chassis_link"/>
     <child link="rear_right_wheel"/>
-    <origin xyz = "-${chassis_length/2 - chassis_length/8} ${chassis_width - 0.1} -${chassis_height/2}" rpy= "${pi/2} 0 0"/>
+    <origin xyz = "-${chassis_length/2 - chassis_length/8} -${wheel_offset_y} -${chassis_height/2}" rpy= "${pi/2} 0 0"/>
     <axis xyz="0 0 1"/>
 </joint>
@@ -136,6 +144,6 @@
     <parent link="chassis_link"/>
     <child link="rear_left_wheel"/>
-    <origin xyz = "-${chassis_length/2 - chassis_length/8} -${chassis_width - 0.1} -${chassis_height/2}" rpy= "-${pi/2} 0 0"/>
-    <axis xyz="0 0 1"/>
+    <origin xyz = "-${chassis_length/2 - chassis_length/8} ${wheel_offset_y} -${chassis_height/2}" rpy= "-${pi/2} 0 0"/>
+    <axis xyz="0 0 -1"/>
 </joint>
 </robot>

File: urdf/s_lidar.xacro (robot description, xacro)
@@ -31,5 +31,5 @@
     <sensor name="laser" type="ray">
         <pose> 0 0 0 0 0 0 </pose>
-        <visualize>true</visualize>
+        <visualize>false</visualize>
         <update_rate>10</update_rate>
         <ray>
